Commit message: attach aruco to anymal bounding box, use base camera as well

File: models/aruco_box/model.sdf.xacro (robot description, xacro)
@@ -1,9 +1,10 @@
 <?xml version="1.0"?>
 <sdf xmlns:xacro="http://www.ros.org/wiki/xacro" version="1.6">
+  <xacro:arg name="aruco_id" default="0"/>
   <xacro:arg name="mass" default="0.5" />
   <xacro:arg name="l_x" default="0.20" />
   <xacro:arg name="l_y" default="0.30" />
   <xacro:arg name="l_z" default="0.10" />
-  <xacro:macro name="aruco_box" params="mass l_x l_y l_z">
+  <xacro:macro name="aruco_box" params="aruco_id mass l_x l_y l_z">
     <model name="aruco_box">
       <link name="box">
@@ -38,5 +39,5 @@
             <contact>
               <ode>
-                <kp>1e4</kp>
+                <kp>${1e5*mass}</kp>
                 <kd>1.0</kd>
               </ode>
@@ -70,5 +71,5 @@
               <uri>model://aruco_marker/materials/scripts</uri>
               <uri>model://aruco_marker/materials/textures</uri>
-              <name>Marker</name>
+              <name>Marker${aruco_id}</name>
             </script>
           </material>
@@ -98,4 +99,4 @@
     </model>
   </xacro:macro>
-  <xacro:aruco_box mass="$(arg mass)" l_x="$(arg l_x)" l_y="$(arg l_y)" l_z="$(arg l_z)"/>
+  <xacro:aruco_box mass="$(arg mass)" aruco_id="$(arg aruco_id)" l_x="$(arg l_x)" l_y="$(arg l_y)" l_z="$(arg l_z)"/>
 </sdf>

Commit message: refactor planner to a separated py pkg && use planner config

File: models/aruco_box/model.sdf.xacro (robot description, xacro)
@@ -6,5 +6,7 @@
   <xacro:arg name="l_y" default="0.30" />
   <xacro:arg name="l_z" default="0.10" />
-  <xacro:macro name="aruco_box" params="aruco_id mass l_x l_y l_z">
+  <xacro:arg name="aruco_x" default="0.0" />
+  <xacro:arg name="aruco_y" default="0.0" />
+  <xacro:macro name="aruco_box" params="aruco_id mass l_x l_y l_z aruco_x aruco_y">
     <model name="aruco_box">
       <link name="box">
@@ -37,4 +39,10 @@
           </geometry>
           <surface>
+            <friction>
+              <ode>
+                <mu>1.0</mu>
+                <mu2>1.0</mu2>
+              </ode>
+            </friction>
             <contact>
               <ode>
@@ -47,5 +55,5 @@
       </link>
       <link name="marker">
-        <pose>0 0 ${l_z} 0 -1.57 0</pose>
+        <pose>${aruco_x} ${aruco_y} ${l_z + 0.001} 0 -1.57 0</pose>
         <inertial>
           <pose>0 0 0 0 0 0</pose>
@@ -99,4 +107,12 @@
     </model>
   </xacro:macro>
-  <xacro:aruco_box mass="$(arg mass)" aruco_id="$(arg aruco_id)" l_x="$(arg l_x)" l_y="$(arg l_y)" l_z="$(arg l_z)"/>
+  <xacro:aruco_box
+    mass="$(arg mass)"
+    aruco_id="$(arg aruco_id)"
+    l_x="$(arg l_x)"
+    l_y="$(arg l_y)"
+    l_z="$(arg l_z)"
+    aruco_x="$(arg aruco_x)"
+    aruco_y="$(arg aruco_y)"
+    />
 </sdf>
